File: electronics/logic board v1/logic_board_v1.kicad_pcb (KiCad board)
At the start: 4 copper layers, 48 x 43.5 mm, 52 parts, among them J1 Screw_Terminal_01x02, J2 SWD, J3 Conn_01x04, J4 USB_B_Micro, Q1 AO3401A, SW1 SW_SPDT, U1 STM32F405RGTx, U2 MP2331HGTL, U3 USBLC6-2SC6, Y1 16MHz

Commit message: Update logic_board_v1.kicad_pcb
Parts:
- removed J3: Conn_01x04, Connector_Molex:Molex_PicoBlade_53048-0410_1x04_P1.25mm_Horizontal
- added C19: 10u, Capacitor_SMD:C_0402_1005Metric, F.Cu at (112.9, 90.4)
- added J10: PWM_Conn, Connector_PinHeader_1.27mm:PinHeader_1x03_P1.27mm_Vertical, F.Cu at (130.5, 75.3)
- added J11: PWM_Conn, Connector_PinHeader_1.27mm:PinHeader_1x03_P1.27mm_Vertical, F.Cu at (127.3, 75.3)
- added J12: PWM_Conn, Connector_PinHeader_1.27mm:PinHeader_1x03_P1.27mm_Vertical, F.Cu at (124.1, 75.3)
- added J13: PWM_Conn, Connector_PinHeader_1.27mm:PinHeader_1x03_P1.27mm_Vertical, F.Cu at (120.8, 75.3)
- added J14: PWM_Conn, Connector_PinHeader_1.27mm:PinHeader_1x03_P1.27mm_Vertical, F.Cu at (117.6, 75.3)
- added J15: PWM_Conn, Connector_PinHeader_1.27mm:PinHeader_1x03_P1.27mm_Vertical, F.Cu at (114.3, 75.3)
- added J16: PWM_Conn, Connector_PinHeader_1.27mm:PinHeader_1x03_P1.27mm_Vertical, F.Cu at (111.1, 75.3)
- added J5: PWM_Conn, Connector_PinHeader_1.27mm:PinHeader_1x03_P1.27mm_Vertical, F.Cu at (146.7, 75.3)
- added J6: PWM_Conn, Connector_PinHeader_1.27mm:PinHeader_1x03_P1.27mm_Vertical, F.Cu at (143.5, 75.3)
- added J7: PWM_Conn, Connector_PinHeader_1.27mm:PinHeader_1x03_P1.27mm_Vertical, F.Cu at (140.3, 75.3)
- added J8: PWM_Conn, Connector_PinHeader_1.27mm:PinHeader_1x03_P1.27mm_Vertical, F.Cu at (137.0, 75.3)
- added J9: PWM_Conn, Connector_PinHeader_1.27mm:PinHeader_1x03_P1.27mm_Vertical, F.Cu at (133.8, 75.3)
- added R14: 10k, Resistor_SMD:R_0402_1005Metric, F.Cu at (146.7, 77.4)
- added R15: 10k, Resistor_SMD:R_0402_1005Metric, F.Cu at (143.5, 77.4)
- added R16: 10k, Resistor_SMD:R_0402_1005Metric, F.Cu at (140.3, 77.4)
- added R17: 10k, Resistor_SMD:R_0402_1005Metric, F.Cu at (137.0, 77.4)
- added R18: 10k, Resistor_SMD:R_0402_1005Metric, F.Cu at (133.8, 77.4)
- added R19: 10k, Resistor_SMD:R_0402_1005Metric, F.Cu at (130.6, 77.4)
- added R20: 10k, Resistor_SMD:R_0402_1005Metric, F.Cu at (127.3, 77.4)
- added R21: 10k, Resistor_SMD:R_0402_1005Metric, F.Cu at (124.1, 77.4)
- added R22: 10k, Resistor_SMD:R_0402_1005Metric, F.Cu at (120.8, 77.4)
- added R23: 10k, Resistor_SMD:R_0402_1005Metric, F.Cu at (117.6, 77.4)
- added R24: 10k, Resistor_SMD:R_0402_1005Metric, F.Cu at (114.4, 77.4)
- added R25: 10k, Resistor_SMD:R_0402_1005Metric, F.Cu at (111.1, 77.4)
- added U4: PCA9685, Package_SO:TSSOP-28_4.4x9.7mm_P0.65mm, F.Cu at (117.4, 86.7)
- D2: footprint Diode_SMD:D_0201_0603Metric -> Diode_SMD:D_SOD-123
- R10, R11, R2, R4, R5, R6, R7, R8, R9: footprint Resistor_SMD:R_0603_1608Metric -> Resistor_SMD:R_0402_1005Metric
- moved J1 41.9 mm to (147.6, 86.9), turned to 90 degrees
- moved H3 20.9 mm to (88.1, 86.9)
- moved R13 19.1 mm to (134.0, 92.2)
- moved D3 18.7 mm to (134.0, 90.6)
- moved R9 17.9 mm to (137.1, 117.6)
- moved L2 17.2 mm to (130.8, 112.8), turned to 180 degrees
- moved R6 16.3 mm to (131.7, 116.2), turned to 180 degrees
- moved R4 15.9 mm to (133.1, 117.4)
- moved SW1 15.8 mm to (108.4, 95.0), turned to -90 degrees
- moved R7 15.6 mm to (135.9, 117.6), turned to 90 degrees
- moved R8 15.1 mm to (138.3, 116.4), turned to 90 degrees
- moved C14 14.9 mm to (134.6, 117.7), turned to -90 degrees
- moved R5 13.9 mm to (133.1, 118.5), turned to 180 degrees
- moved R1 13.4 mm to (114.4, 93.7), turned to 180 degrees
- moved H1 12.9 mm to (161.5, 88.8)
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Connections:
- C16 pad 2: V_OUT -> +3.3V
- L2 pad 2: V_OUT -> +3.3V
- R8 pad 2: V_OUT -> +3.3V
- U1 pad 5: HSE_OUT -> HSE_IN
- U1 pad 6: HSE_IN -> HSE_OUT
- U3 pad 3: USB_D- -> USB_CONN_D+
- U3 pad 4: USB_CONN_D+ -> USB_D+
- U3 pad 6: USB_D+ -> USB_D-
Routing:
- net GND: track 0.00 -> 63.6 mm, vias 0 -> 88
- net PWM0: track 0.00 -> 31.2 mm
- net PWM1: track 0.00 -> 27.7 mm
- net +5V: track 0.00 -> 26.9 mm, vias 0 -> 4
- net PWM2: track 0.00 -> 24.2 mm
- net PWM3: track 0.00 -> 20.7 mm
- net PWM4: track 0.00 -> 17.2 mm
- net SWO: track 25.0 -> 9.12 mm
- net BOOT0: track 25.1 -> 9.23 mm
- net USB_D+: track 1.01 -> 16.6 mm
- net Net-(C15-Pad1): track 17.5 -> 1.90 mm
- net USB_D-: track 0.81 -> 14.8 mm
- net PWM5: track 0.00 -> 13.7 mm
- net NRST: track 28.2 -> 16.5 mm, vias 0 -> 2
- net SWCLK: track 19.3 -> 8.08 mm
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- added copper zone on In2.Cu, net +3.3V
- added copper zone on B.Cu, net +8.4V
- added copper zone on F.Cu, net GND
- added copper zone on In1.Cu, net GND
Other:
- board size 48 x 43.5 mm -> 48 x 65.6 mm
- board text added: "3V3"
- board text added: "BOOT"
- board text added: "I2C"
- board text added: "JLCJLCJLCJLC"
- board text added: "RUN"
- board text added: "STATUS"
- board text added: "STM32F4 TEST BOARD | REV 1"
- board text added: "SWD"
- board text added: "USB"
- board text added: "V+"
- board text added: "^__^ (oo)\_______ (__)\ )\/\ ||-----|| || ||"
- board text added: "⇦"

Commit message: Update logic_board_v1.kicad_pcb
Parts:
- removed H1, H2, H3, H4: MountingHole_Pad, MountingHole:MountingHole_3.2mm_M3_Pad_Via
- removed J4: USB_B_Micro, Connector_USB:USB_Micro-AB_Molex_47590-0001
- added J3: USB_B_Mini, Connector_USB:USB_Mini-B_Lumberg_2486_01_Horizontal, F.Cu at (146.7, 96.7)
- J10, J11, J12, J13, J14, J15, J16, J5, J6, J7, J8, J9: footprint Connector_PinHeader_1.27mm:PinHeader_1x03_P1.27mm_Vertical -> Connector_PinHeader_2.54mm:PinHeader_1x03_P2.54mm_Vertical
- J2: footprint Connector_PinHeader_1.27mm:PinHeader_2x05_P1.27mm_Vertical_SMD -> Connector_PinHeader_2.54mm:PinHeader_2x05_P2.54mm_Vertical_SMD
- U1: value STM32F405RGTx -> STM32F405RGT6
- moved D3 30.8 mm to (143.0, 120.0)
- moved R13 30.8 mm to (143.0, 121.6)
- moved J1 26.4 mm to (147.7, 113.2)
- moved J2 9.97 mm to (134.9, 87.0)
- moved F1 9.59 mm to (142.2, 111.2), turned to 90 degrees
- moved R12 9.38 mm to (139.0, 93.8), turned to 180 degrees
- moved U4 3.29 mm to (120.7, 86.7)
- moved J5 3.27 mm to (150.0, 75.0)
- moved R14 3.26 mm to (150.0, 77.2)
- moved R25 3.14 mm to (108.0, 77.2)
- moved J16 3.10 mm to (108.0, 75.0)
- moved C19 2.89 mm to (115.8, 89.7)
- moved J6 2.70 mm to (146.2, 75.0)
- moved R15 2.68 mm to (146.2, 77.2)
- moved R24 2.56 mm to (111.8, 77.2)
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Routing:
- net +8.4V: track 21.4 -> 5.67 mm, vias 1 -> 0
- net SWO: track 9.12 -> 22.2 mm
- net +5V: track 26.9 -> 14.2 mm, vias 4 -> 0
- net SWCLK: track 8.08 -> 18.5 mm
- net NRST: track 16.5 -> 24.0 mm
- net SWDIO: track 12.2 -> 19.6 mm
- net USB_CONN_D-: track 9.83 -> 3.98 mm, vias 2 -> 0
- net USB_CONN_D+: track 9.59 -> 4.33 mm
- net PWM11: track 9.13 -> 13.3 mm
- net PWM5: track 13.7 -> 10.8 mm
- net GND: track 63.6 -> 60.9 mm, vias 88 -> 127
- net PWM4: track 17.2 -> 14.9 mm
- net PWM8: track 7.86 -> 5.65 mm
- net Net-(Q1-D): track 3.67 -> 5.75 mm
- net PWM10: track 7.84 -> 9.65 mm
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Other:
- board size 48 x 65.6 mm -> 48 x 63 mm
- board text removed: "I2C"

Commit message: update stm32 board project
Parts:
- added C17: 470u, Capacitor_SMD:C_Elec_8x10.2, F.Cu at (147.2, 84.5)
- added C20: 100n, Capacitor_SMD:C_0402_1005Metric, F.Cu at (135.0, 66.3)
- added C21: 100n, Capacitor_SMD:C_0402_1005Metric, F.Cu at (123.0, 66.3)
- added C22: 100n, Capacitor_SMD:C_0402_1005Metric, F.Cu at (146.2, 66.3)
- added C23: 100n, Capacitor_SMD:C_0402_1005Metric, F.Cu at (112.0, 66.3)
- added R5: 1k, Resistor_SMD:R_0402_1005Metric, F.Cu at (129.3, 106.5)
- J1: footprint TerminalBlock_Phoenix:TerminalBlock_Phoenix_PT-1,5-2-3.5-H_1x02_P3.50mm_Horizontal -> TerminalBlock_RND:TerminalBlock_RND_205-00012_1x02_P5.00mm_Horizontal
- R4: value 140k -> 604k
- R7: value 3 -> 20k
- SW1: footprint Button_Switch_SMD:SW_SPDT_PCM12 -> Button_Switch_SMD:SW_SPDT_Shouhan_MSK12C02
- moved J1 0.90 mm to (148.5, 113.0)
Connections:
- U1 pad 42: unconnected-(U1-PA9-Pad42) -> USB_VBUS
- U4 pad 23: unconnected-(U4-~{OE}-Pad23) -> GND
Routing:
- net +8.4V: track 5.67 -> 43.0 mm
- net +5V: track 14.2 -> 21.4 mm
- net USB_VBUS: track 0.00 -> 2.43 mm
- net PWM0: track 31.2 -> 33.6 mm
- net GND: track 60.9 -> 62.4 mm, vias 127 -> 103
Other:
- board text added: ", |`-.__ / ' _/ ****` / } / \ / \ /` \\\ `\ /_\\ `~~~~~``~`"
- board text added: "REV 1"
- board text removed: "STM32F4 TEST BOARD | REV 1"
- board text removed: "^__^ (oo)\_______ (__)\ )\/\ ||-----|| || ||"
