File: electronics/logic board v1/logic_board_v1.kicad_sch (KiCad schematic)
At the start: 48 parts, among them J1 Screw_Terminal_01x02, J2 SWD, J3 Conn_01x04, J4 USB_B_Micro, Q1 AO3401A, SW1 SW_SPDT, U1 STM32F405RGTx, U3 USBLC6-2SC6, Y1 16MHz

Commit message: Update logic_board_v1.kicad_sch
Parts:
- C13, C15, C16, C17: footprint (none) -> Capacitor_SMD:C_0603_1608Metric
- C14, C18: footprint (none) -> Capacitor_SMD:C_0402_1005Metric
- D1, D3: footprint (none) -> LED_SMD:LED_0603_1608Metric
- D2: footprint (none) -> Diode_SMD:D_0201_0603Metric
- R1, R10, R11, R13, R3, R4, R5, R8, R9: footprint (none) -> Resistor_SMD:R_0603_1608Metric
- R12, R2, R6, R7: footprint (none) -> Resistor_SMD:R_0402_1005Metric
Changed lines of the file:
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@@
 			)
 		)
-		(property "Footprint" ""
+		(property "Footprint" "Resistor_SMD:R_0603_1608Metric"
 			(at 110.49 147.32 0)
 			(effects
@@
 			)
 		)
-		(property "Footprint" ""
+		(property "Footprint" "Resistor_SMD:R_0603_1608Metric"
 			(at 92.71 173.99 0)
 			(effects
@@
 			)
 		)
-		(property "Footprint" ""
+		(property "Footprint" "Resistor_SMD:R_0603_1608Metric"
 			(at 97.79 146.05 0)
 			(effects
@@
 			)
 		)
-		(property "Footprint" ""
+		(property "Footprint" "Resistor_SMD:R_0603_1608Metric"
 			(at 95.25 146.05 0)
 			(effects
@@
 			)
 		)
-		(property "Footprint" ""
+		(property "Footprint" "Resistor_SMD:R_0603_1608Metric"
 			(at 170.18 38.1 0)
 			(effects
@@
 			)
 		)
-		(property "Footprint" ""
+		(property "Footprint" "Diode_SMD:D_0201_0603Metric"
 			(at 46.99 21.59 90)
 			(effects
@@
 			)
 		)
-		(property "Footprint" ""
+		(property "Footprint" "Capacitor_SMD:C_0603_1608Metric"
 			(at 68.58 30.48 0)
 			(effects
@@
 			)
 		)
-		(property "Footprint" ""
+		(property "Footprint" "LED_SMD:LED_0603_1608Metric"
 			(at 232.41 30.48 90)
 			(effects
@@
 			)
 		)
-		(property "Footprint" ""
+		(property "Footprint" "Resistor_SMD:R_0603_1608Metric"
 			(at 92.71 30.48 0)
 			(effects
@@
 			)
 		)
-		(property "Footprint" ""
+		(property "Footprint" "Resistor_SMD:R_0402_1005Metric"
 			(at 149.86 34.29 0)
 			(effects
@@
 			)
 		)
-		(property "Footprint" ""
+		(property "Footprint" "Capacitor_SMD:C_0603_1608Metric"
 			(at 153.67 22.86 0)
 			(effects
@@
 			)
 		)
-		(property "Footprint" ""
+		(property "Footprint" "Resistor_SMD:R_0603_1608Metric"
 			(at 92.71 22.86 0)
 			(effects
@@
 			)
 		)
-		(property "Footprint" ""
+		(property "Footprint" "Capacitor_SMD:C_0603_1608Metric"
 			(at 63.5 30.48 0)
 			(effects
@@
 			)
 		)
-		(property "Footprint" ""
+		(property "Footprint" "Resistor_SMD:R_0402_1005Metric"
 			(at 149.86 19.05 0)
 			(effects
@@
 			)
 		)
-		(property "Footprint" ""
+		(property "Footprint" "Resistor_SMD:R_0402_1005Metric"
 			(at 106.68 104.14 0)
 			(effects
@@
 			)
 		)
-		(property "Footprint" ""
+		(property "Footprint" "Capacitor_SMD:C_0603_1608Metric"
 			(at 163.83 30.48 0)
 			(effects
@@
 			)
 		)
-		(property "Footprint" ""
+		(property "Footprint" "Capacitor_SMD:C_0402_1005Metric"
 			(at 77.47 30.48 0)
 			(effects
@@
 			)
 		)
-		(property "Footprint" ""
+		(property "Footprint" "LED_SMD:LED_0603_1608Metric"
 			(at 110.49 140.97 90)
 			(effects
@@
 			)
 		)
-		(property "Footprint" ""
+		(property "Footprint" "Resistor_SMD:R_0603_1608Metric"
 			(at 170.18 30.48 0)
 			(effects
@@
 			)
 		)
-		(property "Footprint" ""
+		(property "Footprint" "Resistor_SMD:R_0402_1005Metric"
 			(at 224.79 64.77 0)
 			(effects
@@
 			)
 		)
-		(property "Footprint" ""
+		(property "Footprint" "Resistor_SMD:R_0603_1608Metric"
 			(at 232.41 35.56 0)
 			(effects
@@
 			)
 		)
-		(property "Footprint" ""
+		(property "Footprint" "Capacitor_SMD:C_0402_1005Metric"
 			(at 118.11 26.67 0)
 			(effects

Commit message: Update logic_board_v1.kicad_sch
Other:
- added sheet Sheet2 (Sheet2.kicad_sch)
Changed lines of the file:
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@@
+		)
+	)
+	(sheet
+		(at 314.96 5.08)
+		(size 297.18 205.74)
+		(exclude_from_sim no)
+		(in_bom yes)
+		(on_board yes)
+		(dnp no)
+		(fields_autoplaced yes)
+		(stroke
+			(width 0.1524)
+			(type solid)
+		)
+		(fill
+			(color 0 0 0 0.0000)
+		)
+		(property "Sheetname" "Sheet2"
+			(at 314.96 4.3684 0)
+			(effects
+				(font
+					(size 1.27 1.27)
+				)
+				(justify left bottom)
+			)
+		)
+		(property "Sheetfile" "Sheet2.kicad_sch"
+			(at 314.96 211.4046 0)
+			(effects
+				(font
+					(size 1.27 1.27)
+				)
+				(justify left top)
+			)
+		)
+		(instances
+			(project "logic_board_v1"
+				(path "/3d6d34b6-2270-42d8-9a55-b901109db90f"
+					(page "2")
+				)
+			)
 		)
 	)

Commit message: Update logic_board_v1.kicad_sch
Parts:
- added H1, H2, H3, H4: MountingHole_Pad, MountingHole:MountingHole_3.2mm_M3_Pad_Via, symbol Mechanical:MountingHole_Pad
- F1: footprint (none) -> Fuse:Fuse_1206_3216Metric
- FB1: footprint (none) -> Inductor_SMD:L_0805_2012Metric
- J1: footprint (none) -> TerminalBlock_Phoenix:TerminalBlock_Phoenix_PT-1,5-2-3.5-H_1x02_P3.50mm_Horizontal
- J2: footprint (none) -> Connector_PinHeader_1.27mm:PinHeader_2x05_P1.27mm_Vertical_SMD
- J3: footprint (none) -> Connector_Molex:Molex_PicoBlade_53048-0410_1x04_P1.25mm_Horizontal
- J4: footprint (none) -> Connector_USB:USB_Micro-AB_Molex_47590-0001
- L1: footprint (none) -> Inductor_SMD:L_0402_1005Metric
- L2: footprint (none) -> Inductor_SMD:L_0603_1608Metric
- R12, R2, R6, R7: footprint Resistor_SMD:R_0402_1005Metric -> Resistor_SMD:R_0603_1608Metric
- SW1: footprint (none) -> Button_Switch_SMD:SW_SPDT_PCM12
- U2: value ~ -> MP2331HGTL; footprint (none) -> Package_TO_SOT_SMD:SOT-583-8
- Y1: footprint (none) -> Crystal:Crystal_SMD_3225-4Pin_3.2x2.5mm
Connections:
- net +3.3V: no longer C10.1, C9.1, L1.2
- net +3.3VA: now also C10.1, C9.1, L1.2
- net GND: now also H1.1, H2.1, H3.1, H4.1
Other:
- removed sheet Sheet2

Commit message: Update logic_board_v1.kicad_sch
Parts:
- removed J3: Conn_01x04, Connector_Molex:Molex_PicoBlade_53048-0410_1x04_P1.25mm_Horizontal, symbol Connector_Generic:Conn_01x04
- D2: footprint Diode_SMD:D_0201_0603Metric -> Diode_SMD:D_SOD-123
- R10, R11, R2, R4, R5, R6, R7, R8, R9: footprint Resistor_SMD:R_0603_1608Metric -> Resistor_SMD:R_0402_1005Metric
Connections:
- net V_OUT is gone; now on net +3.3V: C16.2, L2.2, R8.2
- net HSE_IN: now also U1.5 (PH0); no longer U1.6 (PH1)
- net HSE_OUT: now also U1.6 (PH1); no longer U1.5 (PH0)
- net USB_CONN_D+: now also U3.3 (I/O2); no longer U3.4 (I/O2)
- net USB_D+: now also U3.4 (I/O2); no longer U3.6 (I/O1)
- net USB_D-: now also U3.6 (I/O1); no longer U3.3 (I/O2)
Other:
- added sheet pwm (untitled.kicad_sch)
- moved on the sheet: J4, U3

Commit message: Update logic_board_v1.kicad_sch
Parts:
- removed H1, H2, H3, H4: MountingHole_Pad, MountingHole:MountingHole_3.2mm_M3_Pad_Via, symbol Mechanical:MountingHole_Pad
- removed J4: USB_B_Micro, Connector_USB:USB_Micro-AB_Molex_47590-0001, symbol Connector:USB_B_Micro
- added J3: USB_B_Mini, Connector_USB:USB_Mini-B_Lumberg_2486_01_Horizontal, symbol Connector:USB_B_Mini
- J2: footprint Connector_PinHeader_1.27mm:PinHeader_2x05_P1.27mm_Vertical_SMD -> Connector_PinHeader_2.54mm:PinHeader_2x05_P2.54mm_Vertical_SMD
- U1: value STM32F405RGTx -> STM32F405RGT6
Connections:
- net +5V: now also J3.1 (VBUS)
- net GND: now also J3.5 (GND)
- net USB_CONN_D+: now also J3.3 (D+)
- net USB_CONN_D-: now also J3.2 (D-)
Other:
- sheet pwm: file untitled.kicad_sch -> pwm.kicad_sch

Commit message: update stm32 board project
Parts:
- removed C17: 100u, Capacitor_SMD:C_0603_1608Metric, symbol Device:C_Small
- C1, C2: LCSC (none) -> C23630
- C10: LCSC (none) -> C15195
- C11, C12: LCSC (none) -> C1547
- C13: LCSC (none) -> C59461
- C15: LCSC (none) -> C15849
- C18, C4, C5: LCSC (none) -> C1525
- C3: LCSC (none) -> C19666
- C9: LCSC (none) -> C52923
- D1: LCSC (none) -> C2290
- D2: LCSC (none) -> C8598
- D3: LCSC (none) -> C2286
- J1: footprint TerminalBlock_Phoenix:TerminalBlock_Phoenix_PT-1,5-2-3.5-H_1x02_P3.50mm_Horizontal -> TerminalBlock_RND:TerminalBlock_RND_205-00012_1x02_P5.00mm_Horizontal
- L1: LCSC (none) -> C26443
- L2: LCSC (none) -> C108293
- Q1: LCSC (none) -> C15127
- R1, R3: LCSC (none) -> C23192
- R11: LCSC (none) -> C25900
- R12: LCSC (none) -> C23345
- R13: LCSC (none) -> C20197
- R2: LCSC (none) -> C11930
- R4: value 140k -> 604k; LCSC (none) -> C114151
- R5: value 47k -> 1k; LCSC (none) -> C11930
- R6: LCSC (none) -> C25150
- R7: value 3 -> 20k; LCSC (none) -> C25765
- R8: LCSC (none) -> C25893
- R9: LCSC (none) -> C11788
- SW1: footprint Button_Switch_SMD:SW_SPDT_PCM12 -> Button_Switch_SMD:SW_SPDT_Shouhan_MSK12C02
- U1: LCSC (none) -> C15742
- U2: LCSC (none) -> C6992878
- U3: LCSC (none) -> C7519
- Y1: LCSC (none) -> C13738
Connections:
- net +5V: now also R5.1
- net BUCK_EN: no longer R5.1
- net GND: no longer R5.2
- net USB_VBUS: now reaches U1.42 (PA9)
- net USB_VBUS: now also R5.2
- no-connect marks 46 -> 45
Other:
- moved on the sheet: C13, C18, R4
